File: kicad/MultiPhrom.kicad_sch (KiCad schematic)
At the start: 21 parts, among them J1 Speech Socket, J2 AVR-ISP-6, J3 Micro_SD_Card_Det, U1 ATmega168-20A, U2 74VHC125, U3 AT25SF081-SSHD-X, U4 MIC5504-3.3YM5, Y1 16MHz

Commit message: more examples
Other:
- company: (none) -> BarneyNTD
- title: (none) -> MultiPhrom
Changed lines of the file:
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@@
 (kicad_sch (version 20211123) (generator eeschema)
   (paper "A4")
+  (title_block
+    (title "MultiPhrom")
+    (date "2024-03-25")
+    (company "BarneyNTD")
+  )
   (junction (at 91.44 71.12) (diameter 0) (color 0 0 0 0)
   )
