File: kicad/MultiPhrom.kicad_pcb (KiCad board)
At the start: 2 copper layers, 48.3 x 28.6 mm, 21 parts, among them J1 Speech Socket, J2 AVR-ISP-6, J3 Micro_SD_Card_Det, U1 ATmega168-20A, U2 74VHC125, U3 AT25SF081-SSHD-X, U4 MIC5504-3.3YM5, Y1 16MHz

Commit message: Add sample phroms
Parts:
- moved C4 0.54 mm to (102.1, 95.0)
Routing:
- net GND: track 178.2 -> 177.2 mm
- net VCC: track 66.8 -> 65.9 mm
